Commit message: Clean

File: pfg_description/urdf/turtlebot.urdf.xacro (robot description, xacro)
@@ -12,5 +12,3 @@
   <!-- Body of TurtleBot, with plates, standoffs and Create (including sim sensors) -->
   <turtlebot_body/>
-  <!-- Kinect frames and mounting (includes simulation) -->
-  <turtlebot_kinect/>
 </robot>

File: pfg_description/urdf/turtlebot_hardware.urdf.xacro (robot description, xacro)
@@ -115,31 +115,3 @@
     </link>
   </xacro:macro>
-  <xacro:macro name="turtlebot_standoff_kinect" params="parent number x_loc y_loc z_loc">
-    <joint name="standoff_kinect_${number}_joint" type="fixed">
-      <origin xyz="${x_loc} ${y_loc} ${z_loc}" rpy="0 0 0" />
-      <parent link="${parent}"/>
-      <child link="standoff_kinect_${number}_link" />
-    </joint>
-    <link name="standoff_kinect_${number}_link">
-      <inertial>
-        <mass value="0.001" />
-        <origin xyz="0 0 0" />
-        <inertia ixx="0.0001" ixy="0.0" ixz="0.0"
-          iyy="0.0001" iyz="0.0"
-          izz="0.0001" />
-      </inertial>
-      <visual>
-        <origin xyz=" 0 0 0 " rpy="0 0 0" />
-        <geometry>
-          <mesh filename="package://pfg_description/meshes/68-04556-RA_Kinect_Standoff_Assy.dae" scale="${M_SCALE} ${M_SCALE} ${M_SCALE}"/>
-        </geometry>
-      </visual>
-      <collision>
-        <origin xyz="0.0 0.0 0.0" rpy="0 0 0" />
-        <geometry>
-          <cylinder length="0.008585" radius="0.001111"/>
-        </geometry>
-      </collision>
-    </link>
-  </xacro:macro>
 </robot>
