Commit message: More commentaries... deleted some junk

File: pfg_description/urdf/gazebo.urdf.xacro (robot description, xacro)
@@ -4,61 +4,4 @@
 	xmlns:sensor="http://playerstage.sourceforge.net/gazebo/xmlschema/#sensor"
 	xmlns:xacro="http://ros.org/wiki/xacro" name="turtlebot_gazebo">
-<!-- ASUS Xtion PRO camera for simulation -->
-<!-- gazebo_ros_wge100 plugin is in kt2_gazebo_plugins package -->
-<xacro:macro name="turtlebot_sim_asus_xtion">
-  <gazebo reference="camera_link" >
-    <sensor:camera name="camera" >
-      <imageSize>640 480</imageSize>
-      <imageFormat>R8G8B8</imageFormat>
-      <hfov>62.8</hfov>
-      <nearClip>0.1</nearClip>
-      <farClip>10</farClip>
-      <updateRate>2.0</updateRate>
-      <controller:gazebo_ros_wge100 name="kinect_camera_controller" plugin="libgazebo_ros_wge100.so">
-	<alwaysOn>true</alwaysOn>
-	<updateRate>5000.0</updateRate>
-	<cameraName>camera/rgb</cameraName>
-	<frameName>camera_rgb_optical_frame</frameName>
-	<hackBaseline>0.0</hackBaseline>
-	<CxPrime>320.5</CxPrime>
-	<Cx>320.5</Cx>
-	<Cy>240.5</Cy>
-	<baseline>0.09</baseline>
-	<!-- image_width / (2*tan(hfov_radian /2)) -->
-	<!-- 320 for wide and 772.55 for narrow stereo camera -->
-	<focal_length>525</focal_length>
-	<cameraNamespace>camera/rgb</cameraNamespace>
-	<depthData>true</depthData>
-	<interface:camera name="camera_iface" />
-      </controller:gazebo_ros_wge100>
-    </sensor:camera>
-  </gazebo>
-</xacro:macro>
-<xacro:macro name="turtlebot_sim_kinect">
-  <gazebo reference="camera_link">
-    <sensor:camera name="camera">
-      <imageFormat>R8G8B8</imageFormat>
-      <imageSize>640 480</imageSize>
-      <hfov>60</hfov>
-      <nearClip>0.05</nearClip>
-      <farClip>3</farClip>
-      <updateRate>20</updateRate>
-      <baseline>0.1</baseline>
-      <controller:gazebo_ros_openni_kinect name="kinect_camera_controller" plugin="libgazebo_ros_openni_kinect.so">
-        <alwaysOn>true</alwaysOn>
-        <updateRate>20</updateRate>
-        <imageTopicName>/camera/image_raw</imageTopicName>
-        <pointCloudTopicName>/camera/depth/points</pointCloudTopicName>
-        <cameraInfoTopicName>/camera/camera_info</cameraInfoTopicName>
-        <frameName>camera_depth_optical_frame</frameName>
-        <distortion_k1>0.0</distortion_k1>
-        <distortion_k2>0.0</distortion_k2>
-        <distortion_k3>0.0</distortion_k3>
-        <distortion_t1>0.0</distortion_t1>
-        <distortion_t2>0.0</distortion_t2>
-      </controller:gazebo_ros_openni_kinect>
-    </sensor:camera>
-  </gazebo>
-</xacro:macro>
 <xacro:macro name="turtlebot_sim_imu">
   <gazebo>
